File: Kicad Tutorial/Kicad Tutorial.kicad_sch (KiCad schematic)
At the start: 9 parts, among them SW1 SW_SPDT, U1 ATtiny85V-10P

Commit message: modified
Connections:
- net L_TO_R: now reaches D1.1 (K), R2.1
Changed lines of the file:
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@@
     (company "QUARKTON")
+  )
+  (junction (at 233.68 77.47) (diameter 0) (color 0 0 0 0)
   )
   (junction (at 165.1 73.66) (diameter 0) (color 0 0 0 0)
@@
     (stroke (width 0) (type default))
   )
-  (wire (pts (xy 233.68 73.66) (xy 233.68 80.01))
+  (wire (pts (xy 233.68 73.66) (xy 233.68 77.47))
     (stroke (width 0) (type default))
   )
@@
     (stroke (width 0) (type default))
   )
+  (wire (pts (xy 237.49 77.47) (xy 233.68 77.47))
+    (stroke (width 0) (type default))
+  )
   (wire (pts (xy 194.31 69.85) (xy 194.31 74.93))
     (stroke (width 0) (type default))
@@
   )
   (wire (pts (xy 62.23 92.71) (xy 62.23 95.25))
+    (stroke (width 0) (type default))
+  )
+  (wire (pts (xy 233.68 77.47) (xy 233.68 80.01))
     (stroke (width 0) (type default))
   )
@@
     (effects (font (size 1.27 1.27)) (justify left bottom))
   )
+  (label "L_TO_R" (at 237.49 77.47 0) (fields_autoplaced)
+    (effects (font (size 1.27 1.27)) (justify left bottom))
+  )
   (label "LDR" (at 142.24 74.93 0) (fields_autoplaced)
     (effects (font (size 1.27 1.27)) (justify left bottom))
@@
     (effects (font (size 1.27 1.27)) (justify left bottom))
   )
+  (netclass_flag "" (length 0.05) (shape dot) (at 64.77 77.47 270) (fields_autoplaced)
+    (effects (font (size 1.27 1.27)) (justify right bottom))
+    (property "Netclass" "signal" (at 64.82 76.7715 90)
+      (effects (font (size 1.27 1.27) italic) (justify left) hide)
+    )
+  )
   (symbol (lib_id "power:+3.3V") (at 64.77 59.69 0) (unit 1)
