File: Tutorial 1/Kicad Tutorial.kicad_pcb (KiCad board)
At the start: 2 copper layers, 60 x 60 mm, 9 parts, among them SW1 SW_SPDT, U1 ATtiny85V-10P

Commit message: new updates upto 10
Parts:
- moved R4 3.40 mm to (170.2, 100.7), turned to -90 degrees
Routing:
- net GND: track 0.00 -> 66.0 mm
- net +3.3V: track 0.00 -> 65.2 mm
- net /MIC: track 0.00 -> 29.1 mm
- net /LDR: track 0.00 -> 26.6 mm
- net Net-(BT1--): track 0.00 -> 20.9 mm
- net /L_TO_R: track 0.00 -> 12.3 mm
- net /LED: track 0.00 -> 11.9 mm
Changed lines of the file:
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@@
   )
   (footprint "OptoDevice:R_LDR_5.1x4.3mm_P3.4mm_Vertical" (layer "F.Cu")
-    (at 170.18 104.14 90)
+    (at 170.18 100.74 -90)
     (descr "Resistor, LDR 5.1x3.4mm, see http://yourduino.com/docs/Photoresistor-5516-datasheet.pdf")
     (tags "Resistor LDR5.1x3.4mm")
@@
     (fp_arc (start 3.2 -2.1) (mid 4.280697 0.001697) (end 3.197237 2.101971)
       (stroke (width 0.1) (type solid)) (layer "F.Fab"))
-    (pad "1" thru_hole circle (at 0 0 90) (size 1.5 1.5) (drill 0.8) (layers "*.Cu" "*.Mask")
+    (pad "1" thru_hole circle (at 0 0 270) (size 1.5 1.5) (drill 0.8) (layers "*.Cu" "*.Mask")
       (net 6 "/LDR") (pintype "passive"))
-    (pad "2" thru_hole circle (at 3.4 0 90) (size 1.5 1.5) (drill 0.8) (layers "*.Cu" "*.Mask")
+    (pad "2" thru_hole circle (at 3.4 0 270) (size 1.5 1.5) (drill 0.8) (layers "*.Cu" "*.Mask")
       (net 5 "GND") (pintype "passive"))
     (model "${KICAD6_3DMODEL_DIR}/OptoDevice.3dshapes/R_LDR_5.1x4.3mm_P3.4mm_Vertical.wrl"
@@
   (gr_circle locked (center 152.4 101.6) (end 182.4 101.6)
     (stroke (width 0.1) (type solid)) (fill none) (layer "Edge.Cuts"))
+  (segment (start 132.520914 95.49) (end 154.94 95.49) (width 0.5) (layer "F.Cu") (net 1))
+  (segment (start 164.220914 110.48) (end 164.220914 99.690914) (width 0.5) (layer "F.Cu") (net 1))
+  (segment (start 164.220914 99.690914) (end 160.02 95.49) (width 0.5) (layer "F.Cu") (net 1))
+  (segment (start 160.02 87.39) (end 156.45 87.39) (width 0.5) (layer "F.Cu") (net 1))
+  (segment (start 126.410914 101.6) (end 132.520914 95.49) (width 0.5) (layer "F.Cu") (net 1))
+  (segment (start 154.94 95.49) (end 160.02 95.49) (width 0.5) (layer "F.Cu") (net 1))
+  (segment (start 156.45 87.39) (end 154.94 88.9) (width 0.5) (layer "F.Cu") (net 1))
+  (segment (start 154.94 88.9) (end 154.94 95.49) (width 0.5) (layer "F.Cu") (net 1))
+  (segment (start 153.86 119.38) (end 153.86 109.049086) (width 0.3) (layer "F.Cu") (net 2))
+  (segment (start 153.86 109.049086) (end 146.410914 101.6) (width 0.3) (layer "F.Cu") (net 2))
+  (segment (start 162.56 93.98) (end 162.56 96.52) (width 0.5) (layer "B.Cu") (net 3))
+  (segment (start 160.02 99.06) (end 160.02 101.6) (width 0.5) (layer "B.Cu") (net 3))
+  (segment (start 162.56 96.52) (end 160.02 99.06) (width 0.5) (layer "B.Cu") (net 3))
+  (segment (start 160.02 91.44) (end 162.56 93.98) (width 0.5) (layer "B.Cu") (net 3))
+  (segment (start 160.02 104.14) (end 162.960914 104.14) (width 0.3) (layer "B.Cu") (net 4))
+  (segment (start 162.960914 104.14) (end 169.300914 110.48) (width 0.3) (layer "B.Cu") (net 4))
+  (segment (start 151.86 123.92) (end 152.4 124.46) (width 0.5) (layer "F.Cu") (net 5))
+  (segment (start 177.8 93.98) (end 177.8 101.6) (width 0.5) (layer "F.Cu") (net 5))
+  (segment (start 175.26 91.44) (end 177.8 93.98) (width 0.5) (layer "F.Cu") (net 5))
+  (segment (start 151.86 119.38) (end 151.86 123.92) (width 0.5) (layer "F.Cu") (net 5))
+  (segment (start 152.4 124.46) (end 165.480914 124.46) (width 0.5) (layer "F.Cu") (net 5))
+  (segment (start 165.480914 124.46) (end 171.840914 118.1) (width 0.5) (layer "F.Cu") (net 5))
+  (segment (start 170.18 104.14) (end 175.26 109.22) (width 0.5) (layer "B.Cu") (net 5))
+  (segment (start 175.26 109.22) (end 175.26 116.84) (width 0.5) (layer "B.Cu") (net 5))
+  (segment (start 175.26 104.14) (end 177.8 101.6) (width 0.5) (layer "B.Cu") (net 5))
+  (segment (start 175.26 116.84) (end 174 118.1) (width 0.5) (layer "B.Cu") (net 5))
+  (segment (start 170.18 104.14) (end 175.26 104.14) (width 0.5) (layer "B.Cu") (net 5))
+  (segment (start 174 118.1) (end 171.840914 118.1) (width 0.5) (layer "B.Cu") (net 5))
+  (segment (start 166.760914 110.48) (end 166.760914 104.159086) (width 0.3) (layer "F.Cu") (net 6))
+  (segment (start 172.72 98.2) (end 170.18 100.74) (width 0.3) (layer "F.Cu") (net 6))
+  (segment (start 166.760914 104.159086) (end 170.18 100.74) (width 0.3) (layer "F.Cu") (net 6))
+  (segment (start 172.72 89.93) (end 172.72 98.2) (width 0.3) (layer "F.Cu") (net 6))
+  (segment (start 175.26 87.39) (end 172.72 89.93) (width 0.3) (layer "F.Cu") (net 6))
+  (segment (start 166.760914 118.1) (end 166.760914 115.179086) (width 0.3) (layer "F.Cu") (net 7))
+  (segment (start 166.760914 115.179086) (end 167.64 114.3) (width 0.3) (layer "F.Cu") (net 7))
+  (segment (start 175.26 111.76) (end 175.26 95.49) (width 0.3) (layer "F.Cu") (net 7))
+  (segment (start 167.64 114.3) (end 172.72 114.3) (width 0.3) (layer "F.Cu") (net 7))
+  (segment (start 172.72 114.3) (end 175.26 111.76) (width 0.3) (layer "F.Cu") (net 7))
 )

Commit message: completed
Parts:
- added ?: LOGO, LOGO, F.Cu at (152.4, 81.3)
- added REF**: WEEE-Logo_5.6x8mm_SilkScreen, Symbol:WEEE-Logo_5.6x8mm_SilkScreen, B.Cu at (167.6, 91.4)
- added REF**: CE-Logo_11.2x8mm_SilkScreen, Symbol:CE-Logo_11.2x8mm_SilkScreen, B.Cu at (137.2, 114.3)
- added REF**: KiCad-Logo_6mm_SilkScreen, Symbol:KiCad-Logo_6mm_SilkScreen, B.Cu at (152.4, 81.3)
- added REF**: OSHW-Logo2_14.6x12mm_SilkScreen, Symbol:OSHW-Logo2_14.6x12mm_SilkScreen, B.Cu at (137.2, 101.6)
- moved R2 2.54 mm to (157.5, 91.4)
Other:
- board text added: "ANANDHAKUMAR A"
