File: sensor/sensor.kicad_sch (KiCad schematic)
At the start: 2 parts, among them U1 ATtiny3216-S

Commit message: update
Parts:
- added C1, C2, C3: 1 uF, fab:C_1206, symbol fab:C_1206
- added J1: Conn_01x06_Pin, symbol Connector:Conn_01x06_Pin
- added J2: PinHeader_02x02_P2.54mm_Vertical_SMD, fab:PinHeader_02x02_P2.54mm_Vertical_SMD, symbol fab:PinHeader_02x02_P2.54mm_Vertical_SMD
- added JP1, JP2: Jumper_1206, fab:Jumper_1206, symbol fab:Jumper_1206
- added R1, R2: 499, fab:R_1206, symbol fab:R_1206
- added R10, R7, R8, R9: 1mΩ, fab:R_1206, symbol fab:R_1206
- added R3: 100, fab:R_1206, symbol fab:R_1206
- added R4, R5, R6: 10k, fab:R_1206, symbol fab:R_1206
- added S1: 482016514001, 482016514001:WS-ENTV_4820XX514001, symbol 482016514001:482016514001
- D2: value LED_RABG -> LED_RGB
Connections:
- net at D2.1 (RK): now also R1.2
- net PWR_5V: now reaches D2.2 (A)
- net PWR_5V: now also U1.1 (VCC), C3.1, J1.3 (Pin_3), J2.2 (Pin_2), JP2.1 (A), JP2.2 (B), R4.1, R5.1, R6.1
- net at D2.3 (BK): now also R3.2
- net at D2.4 (GK): now also R2.2
- net SDL: now reaches U1.10 (PB1)
- net SDL: now also J2.1 (Pin_1)
- net SCL: now reaches U1.11 (PB0)
- net SCL: now also J2.4 (Pin_4)
- net L1: now reaches U1.12 (PC0)
- net L1: now also R1.1
- net L2: now reaches U1.13 (PC1)
- net L2: now also R2.1
- net L3: now reaches U1.14 (PC2)
- net L3: now also R3.1
- net SWITCH: now reaches U1.15 (PC3)
- net SWITCH: now also R6.2, S1.1
- net UPDI: now reaches U1.16 (~{RESET}/PA0)
- net UPDI: now also J1.2 (Pin_2)
- net A: now reaches U1.17 (PA1)
- net A: now also C2.1, R4.2, S1.A
- net B: now reaches U1.18 (PA2)
- net B: now also C1.1, R5.2, S1.B
- net GND: now reaches U1.20 (GND)
- net GND: now also J2.3 (Pin_3), JP1.1 (A), JP1.2 (B)
- net Pad4: now reaches U1.4 (PA6)
- net Pad4: now also R10.1
- net Pad1: now reaches U1.5 (PA7)
- net Pad1: now also R7.1
- net Pad2: now reaches U1.6 (PB5)
- net Pad2: now also R8.1
- net Pad3: now reaches U1.7 (PB4)
- net Pad3: now also R9.1
- net RX: now reaches U1.8 (PB3)
- net RX: now also J1.4 (Pin_4)
- net TX: now reaches U1.9 (PB2)
- net TX: now also J1.5 (Pin_5)
- new net PWR_GND: C1.2, C2.2, C3.2, J1.1 (Pin_1), R10.2, R7.2, R8.2, R9.2, S1.2, S1.C
- no-connect marks 0 -> 4
Other:
- note added: "ATTINY 3216"
- note added: "HEADER PIN"
- note added: "JUMPER RESISTOR"
- note added: "RGB LED"
- note added: "ROTARY ENCODER"
- note added: "TO DEBOUNCE"
- note added: "TOUCH PADS"
- note added: "UPDI"
- moved on the sheet: D2, U1
